File: fritzen-pro-micro/fritzen-pro-micro.kicad_pcb (KiCad board)
At the start: 2 copper layers, 3 parts, among them J1 Conn_01x12_Pin, J2 Conn_01x12_Pin, J3 Conn_01x22_Pin

Commit message: Started layouting
Parts:
- added G***: LOGO, Logo:logo-fritzenlab-pequeno, B.Cu at (64.2, 49.7)
Connections:
- net D0-RX1 renamed D0-RXI
- net D1-TX0 renamed D1-TXO
- J3 pad 10: D8 -> D9-A8
- J3 pad 11: D9-A8 -> VIN
- J3 pad 12: VIN -> GND
- J3 pad 3: GND -> D2
- J3 pad 4: D2 -> D3
- J3 pad 5: D3 -> D4-A6
- J3 pad 6: D4-A6 -> D5
- J3 pad 7: D5 -> D6-A7
- J3 pad 8: D6-A7 -> D7
- J3 pad 9: D7 -> D8
Routing:
- net VIN: track 0.00 -> 49.9 mm
- net GND: track 0.00 -> 46.6 mm
- net RESET: track 0.00 -> 45.6 mm
- net 5V: track 0.00 -> 43.8 mm
- net A3: track 0.00 -> 43.0 mm
- net A2: track 0.00 -> 42.0 mm
- net A1: track 0.00 -> 40.8 mm
- net A0: track 0.00 -> 39.6 mm
- net D10: track 0.00 -> 35.3 mm
- net D16-MOSI: track 0.00 -> 35.3 mm
- net D15-SCK: track 0.00 -> 35.1 mm
- net D14-MISO: track 0.00 -> 35.0 mm
- net D2: track 0.00 -> 8.11 mm
- net D9-A8: track 0.00 -> 7.99 mm
- net D8: track 0.00 -> 7.99 mm
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Other:
- board outline added: 25.1 x 57.1 mm
- board text added: "Fritzen Pro Micro"
- board text added: "FritzenLab.com.br Loja.FritzenLab.com.br"

Commit message: edited PCB
Parts:
- G***: moved to F.Cu
- J3: moved to B.Cu
- moved G*** 28.6 mm to (68.7, 77.9), turned to -90 degrees
- turned J3 to 180 degrees
Routing:
- net D10: track 35.3 -> 44.0 mm
- net D15-SCK: track 35.1 -> 42.8 mm
- net D14-MISO: track 35.0 -> 42.2 mm
- net D16-MOSI: track 35.3 -> 41.8 mm
- net GND: track 46.6 -> 42.4 mm
- net A0: track 39.6 -> 42.3 mm
- net VIN: track 49.9 -> 51.6 mm
- net 5V: track 43.8 -> 44.6 mm
- net A1: track 40.8 -> 41.6 mm
Other:
- board size 25.1 x 57.1 mm -> 25 x 57.1 mm
- board text added: "D1-TX |D0-RX |D2 |D3 |D4-A6 |D5 |D6-A7 |D7"

Commit message: finished design, generated gerber
Other:
- board text added: "5V"
- board text added: "A0"
- board text added: "A1"
- board text added: "A2"
- board text added: "A3"
- board text added: "Arduino Pro micro clone from Aliexpress"
- board text added: "D0-RX"
- board text added: "D1-TX"
- board text added: "D10"
- board text added: "D14-MISO"
- board text added: "D15-SCK"
- board text added: "D16-MOSI"
- board text added: "D2"
- board text added: "D3"
- board text added: "D4-A6"
- board text added: "D5"
- board text added: "D6-A7"
- board text added: "D7"
- board text added: "D8"
- board text added: "D9-A8"
- board text added: "GND"
- board text added: "RESET"
- board text added: "VIN"
- board text removed: "D1-TX |D0-RX |D2 |D3 |D4-A6 |D5 |D6-A7 |D7"
